File: hardware/kicad/Główny projekt/ZEGAR ESP32.kicad_sch (KiCad schematic)
At the start: 48 parts, among them Q13 IRLZ44N, Q14 IRLZ44N, Q15 BC547, Q16 BC557, U1 ESP32-WROOM-32D, U12 ESP32-C3-WROOM-02, U13 TC4427xOA, U14 ESP32-C3-WROOM-02, U15 ESP32-C3-WROOM-02, U16 IR2110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

Commit message: 1.33 CLEAN 4
Parts:
- removed U15: ESP32-C3-WROOM-02, RF_Module:ESP32-C3-WROOM-02, symbol RF_Module:ESP32-C3-WROOM-02
- removed U17: CC430F5133xRGZ, Package_DFN_QFN:VQFN-48-1EP_7x7mm_P0.5mm_EP4.1x4.1mm_ThermalVias, symbol MCU_Texas_MSP430:CC430F5133xRGZ
Connections:
- net I2S_DATA: now also U1.13 (IO14); no longer U1.23 (IO15)
- net PMS-RX: now reaches U1.6 (IO34)
- net UART1 RX renamed PMS-TX
- net UART1 TX rezystor 10k pull-down: no longer names the net of U1.14 (IO12)
Other:
- note added: "Przetwornica V1"
- note added: "Przetwornica V2"
- note removed: "CS=3 SCK=6 MOSI=7 MISO=10 GDO0=1 GDO2=0"
