File: hardware/kicad/Główny projekt/ZEGAR ESP32.kicad_sch (KiCad schematic)
At the start: 46 parts, among them Q13 IRLZ44N, Q14 IRLZ44N, Q15 BC547, Q16 BC557, U1 ESP32-WROOM-32D, U12 ESP32-C3-WROOM-02, U13 TC4427xOA, U14 ESP32-C3-WROOM-02, U16 IR2110

Commit message: v2.2 BEZ TESTU
Parts:
- added C15, C16, C19: 100nF, symbol Device:C
- added C17: 100uF, symbol Device:C_Polarized
- added C18: 22uF, symbol Device:C_Polarized
- added C20, C21, C22, C29: 100nF, Capacitor_SMD:C_01005_0402Metric, symbol Device:C
- added C23, C24: 100p, symbol Device:C
- added C25, C26: 12p, symbol Device:C
- added C27, C28: 100n, symbol Device:C
- added D168, D169, D170: D_TVS, Diode_SMD:D_SOD-523, symbol Device:D_TVS
- added D171: D_Schottky, Diode_SMD:D_SOD-323, symbol Device:D_Schottky
- added D172: LED 5V, symbol Device:LED
- added D173: LED 3.3V, symbol Device:LED
- added D175: LED, symbol Device:LED
- added J1: USB_C_Receptacle_USB2.0_16P, symbol Connector:USB_C_Receptacle_USB2.0_16P
- added J2, J3: Conn_01x19_Male, Connector_PinHeader_2.54mm:PinHeader_1x19_P2.54mm_Vertical, symbol Connector:Conn_01x19_Male
- added Q19, Q20: MMSS8050-H-TP, digikey-footprints:SOT-23-3, symbol dk_Transistors-Bipolar-BJT-Single:MMSS8050-H-TP
- added R100: 5.1k, symbol Device:R
- added R101: 5.1K, symbol Device:R
- added R102, R106, R107: 10K, Resistor_SMD:R_01005_0402Metric, symbol Device:R
- added R103, R110: 100k, symbol Device:R
- added R104: 2K, symbol Device:R
- added R105: 1.5K, symbol Device:R
- added R108, R109: 22, symbol Device:R
- added R111: 10k, symbol Device:R
- added R113: 501, symbol Device:R
- added R114: R, symbol Device:R
- added SW1, SW2, SW3: SW_Push, Button_Switch_SMD:SW_SPST_B3S-1000, symbol Switch:SW_Push
- added U15: AZ1084-3.3, symbol Regulator_Linear:AZ1084-3.3
- added U17: CH340C, Package_SO:SOIC-16_3.9x9.9mm_P1.27mm, symbol Interface_USB:CH340C
- added U18: STM32F103C8Tx, Package_QFP:LQFP-48_7x7mm_P0.5mm, symbol MCU_ST_STM32F1:STM32F103C8Tx
- added Y1: 32k768, symbol Device:Crystal
- added Y2: 8M0, symbol Device:Crystal
Connections:
- net +5V: no longer U1.2 (VDD)
- net BUZZER_PIN: now also U1.24 (IO2); no longer U1.31 (IO19)
- net GND: now also C15.2, C16.2, C17.2, C18.2, C19.2, C20.1, C21.1, C22.2, C23.2, C24.2, C25.2, C26.2, C27.1, C28.1, C29.1, D168.1 (A1), D169.1 (A1), D170.1 (A1), D172.1 (K), D173.1 (K), J1.A1 (GND), J1.A12 (GND), J1.B1 (GND), J1.B12 (GND), J1.S1 (SHIELD), J2.14 (Pin_14), J3.1 (Pin_1), J3.7 (Pin_7), R100.2, R101.2, SW1.1, SW2.1, SW3.1, U15.1 (GND), U17.1 (GND), U18.23 (VSS), U18.35 (VSS), U18.47 (VSS), U18.8 (VSSA)
- net IO0: now reaches U1.25 (IO0)
- net IO0: now also C20.2, J3.14 (Pin_14), Q20.3 (C), SW1.2
- net EN: now reaches U1.3 (EN)
- net EN: now also C21.2, C22.1, J2.2 (Pin_2), Q19.3 (C), R102.2, SW2.2
- net RXD0: now reaches U1.34 (RXD0/IO3)
- net RXD0: now also J3.5 (Pin_5), U17.2 (TXD)
- net TXD0: now reaches U1.35 (TXD0/IO1)
- net TXD0: now also J3.4 (Pin_4), U17.3 (RXD)
- net GUT_RX: now reaches U1.7 (IO35)
- net DHT_PIN renamed TOUCH_PAD
- net PMS-RX renamed PMS_RX
- new net: C23.1, U18.3 (PC14), Y1.1
- new net: D173.2 (A), R105.1
- new net: R109.1, U18.33 (PA12)
- new net: D168.2 (A2), D171.2 (A), J1.A4 (VBUS), J1.A9 (VBUS), J1.B4 (VBUS), J1.B9 (VBUS)
- new net: J1.A5 (CC1), R100.1
- new net: J1.B5 (CC2), R101.1
- new net: C24.1, U18.4 (PC15), Y1.2
- new net: Q20.1 (B), R107.2
- new net: D175.1 (K), R113.1
- new net: D172.2 (A), R104.1
- new net: C26.1, U18.6 (PD1), Y2.2
- new net: C25.1, U18.5 (PD0), Y2.1
- new net: Q19.1 (B), R106.2
- new net: R108.1, U18.32 (PA11)
- new net: R103.2, U18.44 (BOOT0)
- new net: R110.2, U18.20 (PB2)
- new net: R113.2, U18.34 (PA13)
- new net BOOT0: R103.1
- new net BOOT1: R110.1
- new net CLK: J3.19 (Pin_19)
- new net CMD: J2.18 (Pin_18)
- new net DTR: Q20.2 (E), R106.1, U17.13 (~{DTR})
- new net EXT_3.3V: C15.1, C17.1, C19.1, C27.2, C28.2, D175.2 (A), R105.2, R111.2, R114.2, U1.2 (VDD), U15.2 (VO), U17.16 (VCC), U17.4 (V3), U18.24 (VDD), U18.36 (VDD), U18.48 (VDD), U18.9 (VDDA)
- new net EXT_5V: C16.1, C18.1, D171.1 (K), J2.19 (Pin_19), R104.2, U15.3 (VI)
- new net GUT_TX: U1.31 (IO19)
- new net IO12: J2.13 (Pin_13)
- new net IO13: J2.15 (Pin_15)
- new net IO14: J2.12 (Pin_12)
- new net IO15: J3.16 (Pin_16)
- new net IO16: J3.12 (Pin_12)
- new net IO17: J3.11 (Pin_11)
- new net IO18: J3.9 (Pin_9)
- new net IO19: J3.8 (Pin_8)
- new net IO2: J3.15 (Pin_15)
- new net IO21: J3.6 (Pin_6)
- new net IO22: J3.3 (Pin_3)
- new net IO23: J3.2 (Pin_2)
- new net IO25: J2.9 (Pin_9)
- new net IO26: J2.10 (Pin_10)
- new net IO27: J2.11 (Pin_11)
- new net IO32: J2.7 (Pin_7)
- new net IO33: J2.8 (Pin_8)
- new net IO34: J2.5 (Pin_5)
- new net IO35: J2.6 (Pin_6)
- new net IO4: J3.13 (Pin_13)
- new net IO5: J3.10 (Pin_10)
- new net RESET: C29.2, R114.1, SW3.2, U18.7 (NRST)
- new net RTS: Q19.2 (E), R107.1, U17.14 (~{RTS})
- new net SD0: J3.18 (Pin_18)
- new net SD1: J3.17 (Pin_17)
- new net SD2: J2.16 (Pin_16)
- new net SD3: J2.17 (Pin_17)
- new net SENSOR_VN: J2.4 (Pin_4)
- new net SENSOR_VP: J2.3 (Pin_3)
- new net USBDM: R108.2
- new net USBDP: R109.2, R111.1
- new net USB_DN: D169.2 (A2), J1.A7 (D-), J1.B7 (D-), U17.6 (UD-)
- new net USB_DP: D170.2 (A2), J1.A6 (D+), J1.B6 (D+), U17.5 (UD+)
- new net VDD33: J2.1 (Pin_1), R102.1
- no-connect marks 1 -> 8
Other:
- note added: "Connectors"
- note added: "GNIAZDO USBC ZASILANIE/PROGRAMOWANIE"
- note added: "MIKROKONTROLER ESP32WROOM32D"
- note added: "PROGRAMOWANIE"
- note added: "PROTOTYPY PRZETWORNIC STEROWANYCH Z MCU"
- note added: "PRZETWORNICA 3.3V"
- note added: "PRZYCISKI"
- moved on the sheet: BT1, C1, C10, C11, C12, C13, C14, C2, C3, C4, C5, C6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

Commit message: v2.3 BEZ TESTU - mostek stepper (STM32 0xB0-0xB4, Guition 0x3A/0x3B), kalibracja CAL_MODE, auto-zjazd 30/120/300/600s, czulosc OUT radaru
Nowy modul include/stepper + src/stepper (FIFO, tor prio, cache REF, pending). STM32_Data: hook + sendStepperCmd (0xB1). EsptoGuition: push 0x3B 14B + sub 0x0A-0x0C + HELLO + fix broadcastSnapshots (eco2/tvoc/flags). AppBoot: begin + migracja NVS->flash STM32. platformio.ini: -I include/stepper. Hardware: kicad_sch + backup zip + usuniecie .lck.
Other:
- moved on the sheet: C15, C16, C17, C18, C19, C20, C21, C22, C23, C24, C25, C26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
